Commit message: fix gripper bugs and enlarge gripper pos from [0, 0.085] to [0, 1.57]

File: src/lerobot/robots/bi_arx5/ARX5_SDK/models/X5.urdf (robot description, URDF)
Before this commit: robot X5, 8 links, 7 joints
Links:
- link link6: mass 0.600 -> 0.635

Commit message: add dataset delete function

File: src/lerobot/robots/bi_arx5/ARX5_SDK/models/X5.urdf (robot description, URDF)
Before this commit: robot X5, 8 links, 7 joints
Links:
- link link6: mass 0.635 -> 0.65
